Commit message: Ported to official UR driver

File: herman_description/urdf/helmet_scanner_description.urdf.xacro (robot description, xacro)
@@ -5,10 +5,10 @@
   <joint name="world_joint" type="fixed">
     <parent link="world" />
-    <child link="ur_arm_base_link" />
+    <child link="base_link" />
     <origin xyz="0 0 0" rpy="3.14159 0 0"/>
   </joint>
-  <xacro:ur3_robot prefix="ur_arm_" joint_limited="true"/>
+  <xacro:ur3_robot prefix="" joint_limited="true"/>
   <joint name="UST_bracket_joint" type="fixed">
-    <parent link="ur_arm_tool0" />
+    <parent link="tool0" />
     <child link="UST_bracket_Link" />
     <origin xyz="0 0 0" rpy="0 -1.5707 -1.5707"/>

File: herman_description/urdf/rubiks_description.urdf.xacro (robot description, xacro)
@@ -1,9 +1,12 @@
 <?xml version="1.0"?>
 <robot xmlns:xacro="http://ros.org/wiki/xacro" name="herman">
+  <xacro:arg name="transmission_hw_interface" default="hardware_interface/PositionJointInterface"/>
+  <xacro:include filename="$(find ur_description)/urdf/common.gazebo.xacro" />
+  <xacro:arg name="kinematics_config" default="$(find ur_description)/config/ur3_default.yaml"/>
   <xacro:include filename="$(find ur_description)/urdf/ur3.urdf.xacro" />
   <link name="world" />
   <joint name="world_joint" type="fixed">
     <parent link="world" />
-    <child link="ur_arm_base_link" />
+    <child link="base_link" />
     <origin xyz="0 0 0" rpy="0 0 0"/>
   </joint>
@@ -18,7 +21,7 @@
     <parent link="world" />
     <child link="socket" />
-    <origin xyz="-0.17761 0.18955 0.1952" rpy="0 0 3.14159"/>
+    <origin xyz="-0.17761 0.18955 0.1942" rpy="0 0 3.14159"/>
   </joint>
-  <xacro:ur3_robot prefix="ur_arm_" joint_limited="true"
+  <xacro:ur3_robot prefix="" joint_limited="true"
     shoulder_pan_lower_limit="${-pi}" shoulder_pan_upper_limit="0.0"
     shoulder_lift_lower_limit="${-pi}" shoulder_lift_upper_limit="${pi}"
@@ -26,9 +29,11 @@
     wrist_1_lower_limit="-4.71229" wrist_1_upper_limit="-1.5707"
     wrist_2_lower_limit="${-pi}" wrist_2_upper_limit="${pi}"
-    wrist_3_lower_limit="${-pi}" wrist_3_upper_limit="${pi}"
+    wrist_3_lower_limit="-6" wrist_3_upper_limit="6"
+    transmission_hw_interface="$(arg transmission_hw_interface)"
+    kinematics_file="${load_yaml('$(arg kinematics_config)')}"
   />
   <link name="cube_centre" />
   <joint name="cube_joint" type="fixed">
-    <parent link="ur_arm_tool0" />
+    <parent link="tool0" />
     <child link="cube_centre" />
     <origin xyz="0 0 0.042" rpy="0 -1.5707 -1.5707"/>
