Commit message: Updated rubiks moveit config.  Cleaned up positions and urdf

File: herman_description/urdf/rubiks_description.urdf.xacro (robot description, xacro)
@@ -12,5 +12,5 @@
     <parent link="world" />
     <child link="fixture" />
-    <origin xyz="0.00078 0.28372 0.04" rpy="0 0 5.616"/>
+    <origin xyz="0.00078 0.28372 0.05" rpy="0 0 4.0453"/>
   </joint>
   <link name="socket" />

Commit message: Updated socket position.  Removed front position, too close to singularity

File: herman_description/urdf/rubiks_description.urdf.xacro (robot description, xacro)
@@ -18,7 +18,14 @@
     <parent link="world" />
     <child link="socket" />
-    <origin xyz="-0.17761 0.27087 0.19504" rpy="0 0 3.14159"/>
+    <origin xyz="-0.17761 0.18955 0.1952" rpy="0 0 3.14159"/>
   </joint>
-  <xacro:ur3_robot prefix="ur_arm_" joint_limited="true"/>
+  <xacro:ur3_robot prefix="ur_arm_" joint_limited="true"
+    shoulder_pan_lower_limit="${-pi}" shoulder_pan_upper_limit="0.0"
+    shoulder_lift_lower_limit="${-pi}" shoulder_lift_upper_limit="${pi}"
+    elbow_joint_lower_limit="${-pi}" elbow_joint_upper_limit="0.0"
+    wrist_1_lower_limit="-4.71229" wrist_1_upper_limit="-1.5707"
+    wrist_2_lower_limit="${-pi}" wrist_2_upper_limit="${pi}"
+    wrist_3_lower_limit="${-pi}" wrist_3_upper_limit="${pi}"
+  />
   <link name="cube_centre" />
   <joint name="cube_joint" type="fixed">

Commit message: Updated urdf. Added cube reader and all motions.  Added models and Blender files

File: herman_description/urdf/rubiks_description.urdf.xacro (robot description, xacro)
@@ -5,5 +5,15 @@
   <xacro:arg name="kinematics_config" default="$(find ur_description)/config/ur3_default.yaml"/>
   <xacro:include filename="$(find ur_description)/urdf/ur3.urdf.xacro" />
-  <link name="world" />
+  <link name="world">
+    <visual>
+      <origin xyz="0 0 0" rpy="0 0 1.5707"/>
+      <geometry>
+        <mesh filename="package://herman_description/meshes/table.stl"/>
+      </geometry>
+      <material name="Wood">
+        <color rgba="0.73 0.61 0.37 1.0"/>
+      </material>
+    </visual>
+  </link>
   <joint name="world_joint" type="fixed">
     <parent link="world" />
@@ -11,5 +21,14 @@
     <origin xyz="0 0 0" rpy="0 0 0"/>
   </joint>
-  <link name="fixture" />
+  <link name="fixture">
+    <visual>
+      <geometry>
+        <mesh filename="package://herman_description/meshes/RubiksFixture.stl"/>
+      </geometry>
+      <material name="LightGrey">
+        <color rgba="0.3 0.3 0.3 1.0"/>
+      </material>
+    </visual>
+  </link>
   <joint name="fixture_joint" type="fixed">
     <parent link="world" />
@@ -17,5 +36,14 @@
     <origin xyz="0.00078 0.28372 0.05" rpy="0 0 4.0453"/>
   </joint>
-  <link name="socket" />
+  <link name="socket">
+    <visual>
+      <geometry>
+        <mesh filename="package://herman_description/meshes/RubiksSocket.stl"/>
+      </geometry>
+      <material name="LightGrey">
+        <color rgba="0.3 0.3 0.3 1.0"/>
+      </material>
+    </visual>
+  </link>
   <joint name="socket_joint" type="fixed">
     <parent link="world" />
@@ -33,5 +61,14 @@
     kinematics_file="${load_yaml('$(arg kinematics_config)')}"
   />
-  <link name="cube_centre" />
+  <link name="cube_centre">
+    <visual>
+      <geometry>
+        <mesh filename="package://herman_description/meshes/RubiksEOAT.stl"/>
+      </geometry>
+      <material name="LightGrey">
+        <color rgba="0.3 0.3 0.3 1.0"/>
+      </material>
+    </visual>
+  </link>
   <joint name="cube_joint" type="fixed">
     <parent link="tool0" />
