Commit message: It works!  Should probably put some error-checking into this...

File: herman_description/urdf/date_description.urdf.xacro (robot description, xacro)
@@ -31,3 +31,16 @@
     kinematics_file="${load_yaml('$(arg kinematics_config)')}"
   />
+  <link name="rg2">
+    <visual>
+      <origin xyz="0 0 0" rpy="0 0 0"/>
+      <geometry>
+        <mesh filename="package://herman_description/meshes/rg2.dae"/>
+      </geometry>
+    </visual>
+  </link>
+  <joint name="rg2_joint" type="fixed">
+    <parent link="tool0" />
+    <child link="rg2" />
+    <origin xyz="0 0 0.179" rpy="0 -1.5707 -1.5707"/>
+  </joint>
 </robot>
